Commit message: Fixed avero_sim launch files

File: nodes/avero_sim/urdf/drone_V3.xacro (robot description, xacro)
@@ -12,5 +12,5 @@
                 <origin xyz="0.0 0.0 0.0" rpy="0.0 0.0 1.0472"/>
                 <geometry>
-                    <mesh filename="package://avero_sim/meshes/Nozzle_${position}_V3.stl" scale="1 1 1"/>
+                    <cylinder radius="0.05" length="0.05"/>
                 </geometry>
             </collision>

Commit message: Publish actuib at 100Hz to /command/motor_speed. Run GazeboSim 5x slower. Use exact same k_f as in gymnasium training. MAV OSCILLATES STABLY!

File: nodes/avero_sim/urdf/drone_V3.xacro (robot description, xacro)
@@ -153,5 +153,5 @@
     <xacro:property name="servo_zero_offset" value="0.0" />
     <!-- Rotor Parameters -->
-    <xacro:property name="thrust_constant" value="${6E-05}" />
+    <xacro:property name="thrust_constant" value="${5.749E-05}" />
     <xacro:property name="moment_constant" value="0.016" />
     <xacro:property name="time_constant_up" value="0.0125" />

Commit message: NN node when actions are change in actuator setpoints. Slowed down gazebo actuator speeds to be more realistic.

File: nodes/avero_sim/urdf/drone_V3.xacro (robot description, xacro)
@@ -140,12 +140,12 @@
     <!-- We need to use different gains for the "inner" and "outer" nozzle -->
     <!-- Servo Parameters -->
-    <xacro:property name="p_gain_1st" value="100.0" />
+    <xacro:property name="p_gain_1st" value="50" />
     <xacro:property name="i_gain_1st" value="0.02" />
     <xacro:property name="d_gain_1st" value="0.35" />
-    <xacro:property name="p_gain_2nd" value="100.0" />
+    <xacro:property name="p_gain_2nd" value="50" />
     <xacro:property name="i_gain_2nd" value="0.02" />
     <xacro:property name="d_gain_2nd" value="0.35" />
-    <xacro:property name="c_min" value="-10.0"/>
-    <xacro:property name="c_max" value="10.0"/>
+    <xacro:property name="c_min" value="-0.115"/>
+    <xacro:property name="c_max" value="0.115"/>
     <xacro:property name="i_min" value="-1.0"/>
     <xacro:property name="i_max" value="1.0"/>
@@ -155,6 +155,6 @@
     <xacro:property name="thrust_constant" value="${5.749E-05}" />
     <xacro:property name="moment_constant" value="0.016" />
-    <xacro:property name="time_constant_up" value="0.0125" />
-    <xacro:property name="time_constant_down" value="0.025" />
+    <xacro:property name="time_constant_up" value="0.2816" />
+    <xacro:property name="time_constant_down" value="0.2816" />
     <xacro:property name="rotor_drag_coefficient" value="${8.06428e-05}" />
     <xacro:property name="rolling_moment_coefficient" value="0.000001" />

Commit message: Unsuccessfully deploy NN trained with decent randomization from AveroRL/feature/velocity_error_control

File: nodes/avero_sim/urdf/drone_V3.xacro (robot description, xacro)
@@ -140,8 +140,8 @@
     <!-- We need to use different gains for the "inner" and "outer" nozzle -->
     <!-- Servo Parameters -->
-    <xacro:property name="p_gain_1st" value="50" />
+    <xacro:property name="p_gain_1st" value="100" />
     <xacro:property name="i_gain_1st" value="0.02" />
     <xacro:property name="d_gain_1st" value="0.35" />
-    <xacro:property name="p_gain_2nd" value="50" />
+    <xacro:property name="p_gain_2nd" value="100" />
     <xacro:property name="i_gain_2nd" value="0.02" />
     <xacro:property name="d_gain_2nd" value="0.35" />
@@ -155,6 +155,6 @@
     <xacro:property name="thrust_constant" value="${5.749E-05}" />
     <xacro:property name="moment_constant" value="0.016" />
-    <xacro:property name="time_constant_up" value="0.2816" />
-    <xacro:property name="time_constant_down" value="0.2816" />
+    <xacro:property name="time_constant_up" value="0.1816" />
+    <xacro:property name="time_constant_down" value="0.1816" />
     <xacro:property name="rotor_drag_coefficient" value="${8.06428e-05}" />
     <xacro:property name="rolling_moment_coefficient" value="0.000001" />

Commit message: These drone_v3.xacro values were used for Gazebo SysID of Nozzle Dynamics. These are more realistic than the really fast ones used before. PID controller won't work with these values.

File: nodes/avero_sim/urdf/drone_V3.xacro (robot description, xacro)
@@ -140,12 +140,12 @@
     <!-- We need to use different gains for the "inner" and "outer" nozzle -->
     <!-- Servo Parameters -->
-    <xacro:property name="p_gain_1st" value="100.0" />
+    <xacro:property name="p_gain_1st" value="150.0" />
     <xacro:property name="i_gain_1st" value="0.02" />
-    <xacro:property name="d_gain_1st" value="0.35" />
-    <xacro:property name="p_gain_2nd" value="100.0" />
+    <xacro:property name="d_gain_1st" value="20" />
+    <xacro:property name="p_gain_2nd" value="150.0" />
     <xacro:property name="i_gain_2nd" value="0.02" />
-    <xacro:property name="d_gain_2nd" value="0.35" />
-    <xacro:property name="c_min" value="-10.0"/>
-    <xacro:property name="c_max" value="10.0"/>
+    <xacro:property name="d_gain_2nd" value="20" />
+    <xacro:property name="c_min" value="-1.5"/>
+    <xacro:property name="c_max" value="1.5"/>
     <xacro:property name="i_min" value="-1.0"/>
     <xacro:property name="i_max" value="1.0"/>

Commit message: These drone_v3.xacro values got System ID k_phi = 10Hz +- 4Hz

File: nodes/avero_sim/urdf/drone_V3.xacro (robot description, xacro)
@@ -140,12 +140,12 @@
     <!-- We need to use different gains for the "inner" and "outer" nozzle -->
     <!-- Servo Parameters -->
-    <xacro:property name="p_gain_1st" value="150.0" />
+    <xacro:property name="p_gain_1st" value="100.0" />
     <xacro:property name="i_gain_1st" value="0.02" />
-    <xacro:property name="d_gain_1st" value="20" />
-    <xacro:property name="p_gain_2nd" value="150.0" />
+    <xacro:property name="d_gain_1st" value="3.5" />
+    <xacro:property name="p_gain_2nd" value="100.0" />
     <xacro:property name="i_gain_2nd" value="0.02" />
-    <xacro:property name="d_gain_2nd" value="20" />
-    <xacro:property name="c_min" value="-1.5"/>
-    <xacro:property name="c_max" value="1.5"/>
+    <xacro:property name="d_gain_2nd" value="3.5" />
+    <xacro:property name="c_min" value="-1.0"/>
+    <xacro:property name="c_max" value="1.0"/>
     <xacro:property name="i_min" value="-1.0"/>
     <xacro:property name="i_max" value="1.0"/>

Commit message: Kind of better value for k_omega Gazebo. It's really hard to model 1. order model with this weird time_constant_up/down filter

File: nodes/avero_sim/urdf/drone_V3.xacro (robot description, xacro)
@@ -155,6 +155,6 @@
     <xacro:property name="thrust_constant" value="${5.749E-05}" />
     <xacro:property name="moment_constant" value="0.016" />
-    <xacro:property name="time_constant_up" value="0.0125" />
-    <xacro:property name="time_constant_down" value="0.025" />
+    <xacro:property name="time_constant_up" value="0.35" />
+    <xacro:property name="time_constant_down" value="0.35" />
     <xacro:property name="rotor_drag_coefficient" value="${8.06428e-05}" />
     <xacro:property name="rolling_moment_coefficient" value="0.000001" />
